Commit message: commented ros_gz_brdige

File: hey_agv/urdf/base.xacro (robot description, xacro)
@@ -6,4 +6,5 @@
     <xacro:property name="wheel_radius" value="0.053" />
     <xacro:property name="wheel_length" value="0.05" />
+    <link name="base_footprint" />
     <link name="base_link">
         <visual>
@@ -22,4 +23,9 @@
         </collision>
     </link>
+    <joint name="base_footprint_joint" type="fixed">
+        <parent link="base_link" />
+        <child link="base_footprint" />
+        <origin xyz="0 0 0" rpy="0 0 0"/>
+    </joint>
     <xacro:macro name="wheel_link" params="prefix">
         <link name="${prefix}_wheel_link">
@@ -114,10 +120,10 @@
         <parent link="base_link" />
         <child link="lift_link" />
-        <origin xyz="0 0 0" rpy="0 0 1.5708"/>
-        <limit lower="0.155" upper="0.187" effort="1000.0" velocity="1.0"/>
+        <origin xyz="0 0 0.187" rpy="0 0 1.5708"/>
+        <limit lower="0" upper="0.2" effort="1000.0" velocity="1.0"/>
         <axis xyz="0 0 1" />
     </joint>
     <gazebo reference="base_link">
-        <material>Gazebo/Black</material>
+        <material>Gazebo/Grey</material>
     </gazebo>
     <gazebo reference="right_wheel_link">
@@ -129,5 +135,5 @@
     <gazebo reference="lidar_link_right">
         <material>Gazebo/White</material>
-        <sensor name='gpu_lidar1' type='gpu_lidar'>"
+        <sensor name='gpu_lidar1' type='gpu_lidar'>
             <pose relative_to='lidar_link_right'>0 0 0 0 0 0</pose>
             <topic>lidar1</topic>
@@ -190,5 +196,6 @@
     </gazebo>
     <gazebo>
-        <plugin filename="gz-sim-diff-drive-system" name="gz::sim::systems::DiffDrive">
+        <plugin filename="gz-sim-diff-drive-system"
+                name="gz::sim::systems::DiffDrive">
             <left_joint>base_left_wheel_joint</left_joint>
             <right_joint>base_right_wheel_joint</right_joint>
@@ -198,8 +205,36 @@
             <topic>cmd_vel</topic>
         </plugin>
-        <plugin filename="gz-sim-sensors-system" name="gz::sim::systems::Sensors">
+    </gazebo>
+    <!-- Fix for sensors plugin -->
+    <gazebo>
+        <plugin filename="gz-sim-sensors-system"
+                name="gz::sim::systems::Sensors">
             <render_engine>ogre2</render_engine>
         </plugin>
     </gazebo>
+     <gazebo>
+        <plugin
+            filename="gz-sim-joint-controller-system"
+            name="gz::sim::systems::JointController">
+            <joint_name>lift_base_joint</joint_name>
+            <initial_velocity>0.05</initial_velocity>
+            <topic>lift_cmd</topic>
+        </plugin>
+    </gazebo>
+    <gazebo>
+        <plugin
+            filename="gz-sim-joint-state-publisher-system"
+            name="gz::sim::systems::JointStatePublisher">
+            <topic>joint_states</topic>
+            <joint_name>base_left_wheel_joint</joint_name>
+            <joint_name>base_right_wheel_joint</joint_name>
+            <joint_name>lift_base_joint</joint_name>
+            </plugin>
+    </gazebo>
+    <!-- <plugin
+            filename="gz-sim-joint-state-publisher-system"
+            name="gz::sim::systems::JointStatePublisher">
+            <joint_name>base_left_wheel_joint</joint_name>
+        </plugin> -->
     <!-- <link name="caster_wheel_link">
         <visual>

File: hey_agv/urdf/properties.xacro (robot description, xacro)
@@ -12,4 +12,7 @@
     <material name="silver">
         <color rgba="0.75 0.75 0.75 1" />
+    </material>
+    <material name="red">
+        <color rgba="1 0 0 1" />
     </material>
     <xacro:macro name="box_inertia" params="m l w h xyz rpy">
